Commit message: Added rgb camer of 2k resolution for deep learning

File: turtlebot3/turtlebot3_description/urdf/turtlebot3_burger.gazebo.xacro (robot description, xacro)
@@ -120,3 +120,59 @@
     </sensor>
   </gazebo>
+  <xacro:macro name="camera" params="parent_name sensor_name origin_xyz camera_YAW">
+    <link name='${sensor_name}_camera_link'>
+		<visual>
+			<origin xyz="0 0 0"
+					rpy="0 0 0"/>
+			<geometry>
+                <mesh filename="package://turtlebot3_description/meshes/sensors/webcam.dae" scale="1.0 1.0 1.0"/>
+			</geometry>
+		</visual>
+	</link>
+    <joint name="${sensor_name}_camera_link_joint" type="fixed">
+		<origin rpy="0 0 ${camera_YAW}" xyz="${origin_xyz}"/>
+		<parent link="${parent_name}"/>
+		<child link="${sensor_name}_camera_link"/>
+	</joint>
+    <link name="${sensor_name}_camera_link_frame">
+    </link>
+    <joint name="${sensor_name}_camera_frame_joint" type="fixed">
+        <origin xyz="0.035 0 0" rpy="0 0 0" />
+        <parent link="${sensor_name}_camera_link" />
+        <child link="${sensor_name}_camera_link_frame" />
+        <axis xyz="0 0 0"/>
+    </joint>
+    <gazebo reference="${sensor_name}_camera_link_frame">
+        <sensor type="camera" name="${sensor_name}">
+        <update_rate>10.0</update_rate>
+        <camera name="${sensor_name}_SP">
+            <pose>0 0 0 0 0 0</pose>
+            <horizontal_fov>1.3962634</horizontal_fov>
+            <image>
+            <width>2040</width>
+            <height>2040</height>
+            <format>R8G8B8</format>
+            </image>
+            <clip>
+                <near>0.005</near>
+                <far>20.0</far>
+            </clip>
+        </camera>
+        <plugin name="camera_controller" filename="libgazebo_ros_camera.so">
+            <alwaysOn>true</alwaysOn>
+            <updateRate>0.0</updateRate>
+            <cameraName>${sensor_name}/rgb</cameraName>
+            <imageTopicName>image_raw</imageTopicName>
+            <cameraInfoTopicName>camera_info</cameraInfoTopicName>
+            <frameName>${sensor_name}_camera_link_frame</frameName>
+            <hackBaseline>0.07</hackBaseline>
+            <distortionK1>0.0</distortionK1>
+            <distortionK2>0.0</distortionK2>
+            <distortionK3>0.0</distortionK3>
+            <distortionT1>0.0</distortionT1>
+            <distortionT2>0.0</distortionT2>
+        </plugin>
+        </sensor>
+    </gazebo>
+  </xacro:macro>
 </robot>

File: turtlebot3/turtlebot3_description/urdf/turtlebot3_burger.urdf.xacro (robot description, xacro)
@@ -140,3 +140,4 @@
     </inertial>
   </link>
+  <xacro:camera sensor_name="camera" parent_name="base_link" origin_xyz="0.015 0.0 0.09" camera_YAW="0.0"/>
 </robot>
